Commit message: 整理代码
把没用的删了一些
现在能跑，但是碰撞盒很奇怪，夹爪会和桌子碰撞变形，另外机械臂会被桌子限制住。

File: models/cube_small_pick.urdf (robot description, URDF)
Before this commit: robot cube.urdf, 1 links, 0 joints
Links:
- link baseLink: mass 2 -> 4; geometry collision box size=.04 .04 .04; visual box size=.04 .04 .04

File: models/cube_small_target_pick.urdf (robot description, URDF)
Before this commit: robot cube.urdf, 1 links, 0 joints
Links:
- link baseLink: mass 2 -> 1; geometry visual box size=.04 .04 .04

Commit message: 能夹取，但是夹不住
目前不清楚是什么问题，夹到了但是物体会弹出去。正在考虑调整硬度和摩擦系数。

File: models/cube_small_pick.urdf (robot description, URDF)
Before this commit: robot cube.urdf, 1 links, 0 joints
Links:
- link baseLink: mass 4 -> 1; geometry collision box size=.08 .04 .04; visual box size=.08 .04 .04
